File: hw/supalaminator.kicad_pcb (KiCad board)
At the start: 2 copper layers, 51.6 x 52.3 mm, 7 parts, among them P1 CONN_RELAY, P2 CONN_THERM, P3 CONN_ROTARY

Commit message: Add power source
Parts:
- added P4: CONN_01X02, Pin_Headers:Pin_Header_Straight_1x02, F.Cu at (89.8, 116.2)
Connections:
- ARD1 pad 15: (no net) -> Net-(ARD1-Pad15)
Routing:
- net Net-(ARD1-Pad15): track 0.00 -> 6.80 mm
