File: hw/supalaminator.sch (KiCad schematic (older format))
At the start: 1 part

Commit message: Final hardware schematic
Parts:
- added ARD1: Arduino_Nano, Arduino:Arduino Nano, symbol Arduino_Nano
- added P1: CONN_RELAY, Pin_Headers:Pin_Header_Straight_1x03, symbol CONN_01X03
- added P2: CONN_THERM, Pin_Headers:Pin_Header_Straight_1x05, symbol CONN_01X05
- added P3: CONN_ROTARY, Pin_Headers:Pin_Header_Straight_1x05, symbol CONN_01X05
- added R1, R2: R, Resistors_ThroughHole:Resistor_Horizontal_RM7mm, symbol R
- DS1: renamed from DS?; footprint WC1602A -> Pin_Headers:Pin_Header_Straight_2x08
Connections:
- net GND: now reaches DS1.1 (VSS)
- net GND: now also DS1.5 (R/W), ARD1.14 (GND), P1.2 (P2), P2.5 (P5), P3.5 (P5), R2.2
- net LCD_D4: now reaches DS1.11 (D4)
- net LCD_D4: now also ARD1.28 (D10)
- net LCD_D5: now reaches DS1.12 (D5)
- net LCD_D5: now also ARD1.25 (D7)
- net LCD_D6: now reaches DS1.13 (D6)
- net LCD_D6: now also ARD1.27 (D9)
- net LCD_D7: now reaches DS1.14 (D7)
- net LCD_D7: now also ARD1.26 (D8)
- net +5V: now reaches DS1.2 (VDD)
- net +5V: now also ARD1.12 (5V), P1.1 (P1), P2.4 (P4), P3.4 (P4), R1.1
- net at DS1.3 (VO): now also R1.2, R2.1
- net LCD_RS: now reaches DS1.4 (RS)
- net LCD_RS: now also ARD1.30 (D12)
- net LCD_E: now reaches DS1.6 (E)
- net LCD_E: now also ARD1.29 (D11)
- new net CS: ARD1.23 (D5), P2.2 (P2)
- new net DO: ARD1.22 (D4), P2.1 (P1)
- new net RELAY: ARD1.4 (A0), P1.3 (P3)
- new net ROT_A: ARD1.21 (D3), P3.2 (P2)
- new net ROT_B: ARD1.20 (D2), P3.1 (P1)
- new net SCK: ARD1.24 (D6), P2.3 (P3)
- new net SW: ARD1.5 (A1), P3.3 (P3)
Other:
- moved on the sheet: DS1

Commit message: Add power source
Parts:
- added P4: CONN_01X02, Pin_Headers:Pin_Header_Straight_1x02, symbol CONN_01X02
Connections:
- net GND: now also P4.2 (P2)
- net at ARD1.15 (VIN): now also P4.1 (P1)
Changed lines of the file:
@@
 LIBS:memory
 LIBS:xilinx
+LIBS:special
 LIBS:microcontrollers
 LIBS:dsp
@@
 Wire Wire Line
 	2150 5200 2700 5200
+$Comp
+L CONN_01X02 P4
+U 1 1 57A9B979
+P 2550 5800
+F 0 "P4" H 2550 5950 50  0000 C CNN
+F 1 "CONN_01X02" V 2650 5800 50  0000 C CNN
+F 2 "Pin_Headers:Pin_Header_Straight_1x02" H 2550 5800 60  0001 C CNN
+F 3 "" H 2550 5800 60  0000 C CNN
+	1    2550 5800
+	0    1    1    0
+$EndComp
+Wire Wire Line
+	2600 5600 2600 5300
+Wire Wire Line
+	2600 5300 2700 5300
+$Comp
+L GND #PWR014
+U 1 1 57A9BA3E
+P 2100 5600
+F 0 "#PWR014" H 2100 5350 50  0001 C CNN
+F 1 "GND" H 2105 5427 50  0000 C CNN
+F 2 "" H 2100 5600 50  0000 C CNN
+F 3 "" H 2100 5600 50  0000 C CNN
+	1    2100 5600
+	1    0    0    -1
+$EndComp
+Wire Wire Line
+	2500 5600 2100 5600
 $EndSCHEMATC
